Commit message: add tf2 sample01

File: musashi_description/urdf/musashi_player.urdf (robot description, URDF)
Before this commit: robot musashi_player, 1 links, 0 joints
Links:
- added link map
- link base_link: geometry collision mesh filename=package://musashi_description/meshes/musashi_player.stl scale=0.001 0.001 0.001; visual mesh filename=package://musashi_description/meshes/musashi_player.stl scale=0.001 0.001 0.001
Joints:
- added joint map_to_base: type fixed, parent map, child base_link, origin xyz=0 0 0 rpy=0 0 0

Commit message: mod README(basestation)

File: musashi_description/urdf/musashi_player.urdf (robot description, URDF)
Before this commit: robot musashi_player, 2 links, 1 joints
Links:
- removed link map
- added link foot_print
Joints:
- removed joint map_to_base
- added joint foot_print_to_base_link: type fixed, parent foot_print, child base_link, origin xyz=0 0 0 rpy=0 0 0
